File: probe v2.sch (EAGLE design)
At the start: 12 parts, among them IC1 74AHC1G14DBV

Commit message: First try to make a connection box directly on machine
Parts:
- removed BALL, BALL1, GND, OUT, VCC: (no value), pinhead:PINHD-1X1
- removed IC1: 74AHC1G14DBV, 74xx-little-us:74AHC1G14DBV
- added BALL1G, BALL1S, BALL2G, BALL2S: (no value), pinhead:PINHD-1X1
- added IC2: 74AC00N, 74xx-eu:74AC00N
- added IC3: 74AC14N, 74xx-eu:74AC14N
- added R4: 1k, rcl:R-EU_0207/10
- added TO_LIMITS, TO_MESA: (no value), con-amp:558310-1
- C1: device rcl:C-EUC0805 -> rcl:CPOL-EUE5-10.5
- GREEN, RED: device led:LEDCHIPLED_1206 -> led:LED5MM
- R1: device rcl:R-EU_R0805 -> rcl:R-EU_0207/10
- R2, R3: device rcl:R-EU_M1206 -> rcl:R-EU_0207/10
Connections:
- removed net OUT: GREEN.C, IC1A.O, OUT.1, RED.A
- new net LIMIT_A: TO_MESA.5
- new net LIMIT_X: TO_MESA.2
- new net LIMIT_Y: TO_MESA.3
- new net LIMIT_Z: TO_MESA.4
- new net N$12: TO_MESA.6
- new net N$4: IC2A.I0, IC3A.O
- new net N$5: IC2A.I1, IC3B.O
- new net N$6: BALL2S.1, IC3A.I, R4.1
- new net N$7: IC2A.O, IC2B.I1
- new net PROBE: GREEN.C, IC2B.O, RED.A, TO_MESA.7
- net BALL: now also BALL1S.1, IC3B.I; no longer BALL.1, IC1A.I
- net GND: now also BALL1G.1, BALL2G.1, C1.-, IC2P.GND, IC3P.GND, TO_LIMITS.8, TO_LIMITS.S1, TO_MESA.8, TO_MESA.S1; no longer BALL1.1, C1.2, GND.1, IC1P.GND
- net VCC: now also C1.+, IC2B.I0, IC2P.VCC, IC3P.VCC, R4.2, TO_LIMITS.1, TO_MESA.1; no longer C1.1, IC1P.VCC, VCC.1
Other:
- moved on the sheet: GREEN, R2, R3, RED
